File: mini-motor-controller.kicad_pcb (KiCad board)
At the start: 2 copper layers, 28.2 x 24.5 mm, 39 parts, among them J1 IN, J2 ADC, J3 FPC, J4 MOT, P1 TC2030, U1 AP2204R-3.3, U2 STM32F030F4Px, U3 STSPIN220

Commit message: bumped files
Other:
- board text added: "+ - A"
- board text added: "+ - B"
- board text added: "GND IN 3V3 ADC"
- board text added: "GND SDA SCL VIN INPUT"
